Commit message: Add 3rd camera

File: workspaceRos/src/phantomx/phantomx_description/urdf/phantomx_urdf.xacro (robot description, xacro)
@@ -42,143 +42,77 @@
         <xacro:leg_l xyz="0 0.1034  0.001116" rpy="0 4.7123 3.14159" suffix="lm"/>
         <xacro:leg_l xyz="-0.1248 0.06164  0.001116" rpy="0 4.7123 3.9269908169872414" suffix="lr"/>
-      <xacro:camera2 xyz="0 -0.08164  0.142" rpy="0 0 -1.5707" suffix="right"/>
-      <xacro:camera2 xyz="0 0.08164  0.142" rpy="0 0 1.5707" suffix="left"/>
-	</xacro:macro>
+<!-- <xacro:camera2 xyz="0 -0.08164  0.142" rpy="0 0 -1.5707" suffix="right"/>
+ <xacro:camera2 xyz="0 0.08164  0.142" rpy="0 0 1.5707" suffix="left"/> -->
+ <xacro:camera2 xyz="-0.1 -0.08164  0.142" rpy="0 -0.52 -1.5707" suffix="right"/>
+ <xacro:camera2 xyz="-0.1 0.08164  0.142" rpy="0 -0.52 1.5707" suffix="left"/>
+ <xacro:camera2 xyz="0.125 0  0.142" rpy="0 -0.52 0" suffix="front"/>
+</xacro:macro>
 <xacro:macro name="camera2" params="xyz rpy suffix">
 <joint name="phantomx_camera_${suffix}" type="fixed">
-    <parent link="MP_BODY"/>
-    <child link="camera_${suffix}"/>
-    <origin xyz="${xyz}" rpy="${rpy}" />
+<parent link="MP_BODY"/>
+<child link="camera_${suffix}"/>
+<origin xyz="${xyz}" rpy="${rpy}" />
 </joint>
 <link name="camera_${suffix}">
-  <inertial>
-    <origin xyz="0 0 0" rpy="0 0 0"/>
-    <mass value="0.1"/>
-    <inertia ixx="0.2" ixy="0" ixz="0" iyy="0.2" iyz="0"
-             izz="0.2"/>
-  </inertial>
-  <collision>
-    <origin xyz="0 0 0" rpy="0 0 0"/>
-    <geometry>
-      <box size="0.073000 0.276000 0.072000"/>
-    </geometry>
-  </collision>
-  <visual>
-    <origin xyz="0 0 0" rpy="0 0 0"/>
-    <geometry>
-         <!--<box size="0.073000 0.276000 0.072000"/>-->
-         <mesh filename="package://phantomx_description/meshes/kinect/meshes/kinect.dae" />-->
-    </geometry>
-  </visual>
+<inertial>
+<origin xyz="0 0 0" rpy="0 0 0"/>
+<mass value="0.1"/>
+<inertia ixx="0.2" ixy="0" ixz="0" iyy="0.2" iyz="0"
+        izz="0.2"/>
+</inertial>
+<collision>
+<origin xyz="0 0 0" rpy="0 0 0"/>
+<geometry>
+ <box size="0.073000 0.276000 0.072000"/>
+</geometry>
+</collision>
+<visual>
+<origin xyz="0 0 0" rpy="0 0 0"/>
+<geometry>
+    <!--<box size="0.073000 0.276000 0.072000"/>-->
+    <mesh filename="package://phantomx_description/meshes/kinect/meshes/kinect.dae" />-->
+</geometry>
+</visual>
 </link>
 <gazebo reference="camera_${suffix}">
- <sensor name="camera_{suffix}" type="depth">
-    <update_rate>20</update_rate>
-    <camera>
-      <horizontal_fov>1.047198</horizontal_fov>
-      <image>
-        <width>640</width>
-        <height>480</height>
-        <format>R8G8B8</format>
-      </image>
-      <clip>
-        <near>0.05</near>
-        <far>3</far>
-      </clip>
-    </camera>
-    <plugin name="camera_plugin" filename="libgazebo_ros_openni_kinect.so">
-          <baseline>0.2</baseline>
-          <alwaysOn>true</alwaysOn>
-          <updateRate>0.0</updateRate>
-          <cameraName>camera_${suffix}</cameraName>
-          <imageTopicName>/phantomx/camera_${suffix}/color/image_raw</imageTopicName>
-          <cameraInfoTopicName>/phantomx/camera_${suffix}/color/camera_info</cameraInfoTopicName>
-          <depthImageTopicName>/phantomx/camera_${suffix}/depth/image_raw</depthImageTopicName>
-          <depthImageCameraInfoTopicName>/phantomx/camera_${suffix}/depth/camera_info</depthImageCameraInfoTopicName>
-          <pointCloudTopicName>/phantomx/camera_${suffix}/depth/points</pointCloudTopicName>
-          <frameName>camera_${suffix}</frameName>
-          <pointCloudCutoff>0.5</pointCloudCutoff>
-          <pointCloudCutoffMax>3.0</pointCloudCutoffMax>
-          <distortionK1>0</distortionK1>
-          <distortionK2>0</distortionK2>
-          <distortionK3>0</distortionK3>
-          <distortionT1>0</distortionT1>
-          <distortionT2>0</distortionT2>
-          <CxPrime>0</CxPrime>
-          <Cx>0</Cx>
-          <Cy>0</Cy>
-          <focalLength>0</focalLength>
-          <hackBaseline>0</hackBaseline>
-        </plugin>
-  </sensor>
-</gazebo>
-</xacro:macro>
- <xacro:macro name="camera2" params="xyz rpy suffix">
-<joint name="phantomx_camera_${suffix}" type="fixed">
-    <parent link="MP_BODY"/>
-    <child link="camera_${suffix}"/>
-    <origin xyz="${xyz}" rpy="${rpy}" />
-</joint>
-<link name="camera_${suffix}">
-  <inertial>
-    <origin xyz="0 0 0" rpy="0 0 0"/>
-    <mass value="0.1"/>
-    <inertia ixx="0.2" ixy="0" ixz="0" iyy="0.2" iyz="0"
-             izz="0.2"/>
-  </inertial>
-  <collision>
-    <origin xyz="0 0 0" rpy="0 0 0"/>
-    <geometry>
-      <box size="0.073000 0.276000 0.072000"/>
-    </geometry>
-  </collision>
-  <visual>
-    <origin xyz="0 0 0" rpy="0 0 0"/>
-    <geometry>
-         <!--<box size="0.073000 0.276000 0.072000"/>-->
-         <mesh filename="package://phantomx_description/meshes/kinect/meshes/kinect.dae" />-->
-    </geometry>
-  </visual>
-</link>
-<gazebo reference="camera_${suffix}">
- <sensor name="camera_{suffix}" type="depth">
-    <update_rate>20</update_rate>
-    <camera>
-      <horizontal_fov>1.047198</horizontal_fov>
-      <image>
-        <width>640</width>
-        <height>480</height>
-        <format>R8G8B8</format>
-      </image>
-      <clip>
-        <near>0.05</near>
-        <far>3</far>
-      </clip>
-    </camera>
-    <plugin name="camera_plugin" filename="libgazebo_ros_openni_kinect.so">
-          <baseline>0.2</baseline>
-          <alwaysOn>true</alwaysOn>
-          <updateRate>0.0</updateRate>
-          <cameraName>camera_${suffix}</cameraName>
-          <imageTopicName>/phantomx/camera_${suffix}/color/image_raw</imageTopicName>
-          <cameraInfoTopicName>/phantomx/camera_${suffix}/color/camera_info</cameraInfoTopicName>
-          <depthImageTopicName>/phantomx/camera_${suffix}/depth/image_raw</depthImageTopicName>
-          <depthImageCameraInfoTopicName>/phantomx/camera_${suffix}/depth/camera_info</depthImageCameraInfoTopicName>
-          <pointCloudTopicName>/phantomx/camera_${suffix}/depth/points</pointCloudTopicName>
-          <frameName>camera_${suffix}</frameName>
-          <pointCloudCutoff>0.5</pointCloudCutoff>
-          <pointCloudCutoffMax>3.0</pointCloudCutoffMax>
-          <distortionK1>0</distortionK1>
-          <distortionK2>0</distortionK2>
-          <distortionK3>0</distortionK3>
-          <distortionT1>0</distortionT1>
-          <distortionT2>0</distortionT2>
-          <CxPrime>0</CxPrime>
-          <Cx>0</Cx>
-          <Cy>0</Cy>
-          <focalLength>0</focalLength>
-          <hackBaseline>0</hackBaseline>
-        </plugin>
-  </sensor>
+<sensor name="camera_{suffix}" type="depth">
+<update_rate>20</update_rate>
+<camera>
+ <horizontal_fov>1.047198</horizontal_fov>
+ <image>
+   <width>640</width>
+   <height>480</height>
+   <format>R8G8B8</format>
+ </image>
+ <clip>
+   <near>0.05</near>
+   <far>10</far>
+ </clip>
+</camera>
+<plugin name="camera_plugin" filename="libgazebo_ros_openni_kinect.so">
+     <baseline>0.2</baseline>
+     <alwaysOn>true</alwaysOn>
+     <updateRate>0.0</updateRate>
+     <cameraName>camera_${suffix}</cameraName>
+     <imageTopicName>/phantomx/camera_${suffix}/color/image_raw</imageTopicName>
+     <cameraInfoTopicName>/phantomx/camera_${suffix}/color/camera_info</cameraInfoTopicName>
+     <depthImageTopicName>/phantomx/camera_${suffix}/depth/image_raw</depthImageTopicName>
+     <depthImageCameraInfoTopicName>/phantomx/camera_${suffix}/depth/camera_info</depthImageCameraInfoTopicName>
+     <pointCloudTopicName>/phantomx/camera_${suffix}/depth/points</pointCloudTopicName>
+     <frameName>camera_${suffix}</frameName>
+     <pointCloudCutoff>0.1</pointCloudCutoff>
+     <pointCloudCutoffMax>2.0</pointCloudCutoffMax>
+     <distortionK1>0</distortionK1>
+     <distortionK2>0</distortionK2>
+     <distortionK3>0</distortionK3>
+     <distortionT1>0</distortionT1>
+     <distortionT2>0</distortionT2>
+     <CxPrime>0</CxPrime>
+     <Cx>0</Cx>
+     <Cy>0</Cy>
+     <focalLength>0</focalLength>
+     <hackBaseline>0</hackBaseline>
+   </plugin>
+</sensor>
 </gazebo>
 </xacro:macro>
@@ -365,22 +299,4 @@
         <gazebo reference="tibia_${suffix}">
             <material>Gazebo/Grey</material>
-        </gazebo>
-        <gazebo reference="MP_BODY">
-          <gravity>true</gravity>
-          <sensor name="imu_sensor" type="imu">
-            <always_on>true</always_on>
-            <update_rate>100</update_rate>
-            <visualize>true</visualize>
-            <plugin filename="libgazebo_ros_imu_sensor.so" name="imu_plugin">
-              <topicName>imu</topicName>
-              <bodyName>MP_BODY</bodyName>
-              <updateRateHZ>10.0</updateRateHZ>
-              <gaussianNoise>0.0</gaussianNoise>
-              <xyzOffset>0 0 0</xyzOffset>
-              <rpyOffset>0 0 0</rpyOffset>
-              <frameName>imu_link</frameName>
-            </plugin>
-            <pose>0 0 0 0 0 0</pose>
-          </sensor>
         </gazebo>
     </xacro:macro>
@@ -539,6 +455,5 @@
           </ray>
           <plugin name="lidar" filename="libgazebo_ros_laser.so">
-            <topicName>lidar</topicName>
-            <frameName>lidar_link</frameName>
+            <topicName>phantomx/lidar</topicName>
           </plugin>
         </sensor>

Commit message: remove left right cameras and lights, add support for front camera

File: workspaceRos/src/phantomx/phantomx_description/urdf/phantomx_urdf.xacro (robot description, xacro)
@@ -44,76 +44,101 @@
 <!-- <xacro:camera2 xyz="0 -0.08164  0.142" rpy="0 0 -1.5707" suffix="right"/>
  <xacro:camera2 xyz="0 0.08164  0.142" rpy="0 0 1.5707" suffix="left"/> -->
- <xacro:camera2 xyz="-0.1 -0.08164  0.142" rpy="0 -0.25 -1.5707" suffix="right"/>
- <xacro:camera2 xyz="-0.1 0.08164  0.142" rpy="0 -0.25 1.5707" suffix="left"/>
- <xacro:camera2 xyz="0.125 0  0.142" rpy="0 -0.25 0" suffix="front"/>
+        <!--xacro:camera2 xyz="-0.1 -0.08164  0.142" rpy="0 -0.25 -1.5707" suffix="right"/>
+        <xacro:camera2 xyz="-0.1 0.08164  0.142" rpy="0 -0.25 1.5707" suffix="left"/-->
+        <xacro:camera2 xyz="0.125 0  0.142" rpy="0 -0.25 0" suffix="front"/>
+        <joint name="phantomx_camera_base_front" type="fixed">
+            <parent link="MP_BODY"/>
+            <child link="camera_base_front"/>
+            <origin xyz="0.100 0 0.060" rpy="0 0 0" />
+        </joint>
+        <link name="camera_base_front">
+            <inertial>
+                <origin xyz="0 0 0" rpy="0 0 0"/>
+                <mass value="0.001"/>
+                <inertia ixx="0.01" ixy="0" ixz="0" iyy="0.01" iyz="0"
+                    izz="0.01"/>
+            </inertial>
+            <collision>
+                <origin xyz="0 0 0" rpy="0 0 0"/>
+                <geometry>
+                    <box size="0.073000 0.276000 0.072000"/>
+                </geometry>
+            </collision>
+            <visual>
+                <origin xyz="0 0 0" rpy="0 0 0"/>
+                <geometry>
+                    <box size="0.03 0.05 0.070 "/>
+                </geometry>
+            </visual>
+        </link>
 </xacro:macro>
 <xacro:macro name="camera2" params="xyz rpy suffix">
-<joint name="phantomx_camera_${suffix}" type="fixed">
-<parent link="MP_BODY"/>
-<child link="camera_${suffix}"/>
-<origin xyz="${xyz}" rpy="${rpy}" />
-</joint>
-<link name="camera_${suffix}">
-<inertial>
-<origin xyz="0 0 0" rpy="0 0 0"/>
-<mass value="0.1"/>
-<inertia ixx="0.2" ixy="0" ixz="0" iyy="0.2" iyz="0"
-        izz="0.2"/>
-</inertial>
-<collision>
-<origin xyz="0 0 0" rpy="0 0 0"/>
-<geometry>
- <box size="0.073000 0.276000 0.072000"/>
-</geometry>
-</collision>
-<visual>
-<origin xyz="0 0 0" rpy="0 0 0"/>
-<geometry>
-    <!--<box size="0.073000 0.276000 0.072000"/>-->
-    <mesh filename="package://phantomx_description/meshes/kinect/meshes/kinect.dae" />-->
-</geometry>
-</visual>
-</link>
-<gazebo reference="camera_${suffix}">
-<sensor name="camera_{suffix}" type="depth">
-<update_rate>20</update_rate>
-<camera>
- <horizontal_fov>1.047198</horizontal_fov>
- <image>
-   <width>640</width>
-   <height>480</height>
-   <format>R8G8B8</format>
- </image>
- <clip>
-   <near>0.05</near>
-   <far>10</far>
- </clip>
-</camera>
-<plugin name="camera_plugin" filename="libgazebo_ros_openni_kinect.so">
-     <baseline>0.2</baseline>
-     <alwaysOn>true</alwaysOn>
-     <updateRate>0.0</updateRate>
-     <cameraName>camera_${suffix}</cameraName>
-     <imageTopicName>/phantomx/camera_${suffix}/color/image_raw</imageTopicName>
-     <cameraInfoTopicName>/phantomx/camera_${suffix}/color/camera_info</cameraInfoTopicName>
-     <depthImageTopicName>/phantomx/camera_${suffix}/depth/image_raw</depthImageTopicName>
-     <depthImageCameraInfoTopicName>/phantomx/camera_${suffix}/depth/camera_info</depthImageCameraInfoTopicName>
-     <pointCloudTopicName>/phantomx/camera_${suffix}/depth/points</pointCloudTopicName>
-     <frameName>camera_${suffix}</frameName>
-     <pointCloudCutoff>0.1</pointCloudCutoff>
-     <pointCloudCutoffMax>2.0</pointCloudCutoffMax>
-     <distortionK1>0</distortionK1>
-     <distortionK2>0</distortionK2>
-     <distortionK3>0</distortionK3>
-     <distortionT1>0</distortionT1>
-     <distortionT2>0</distortionT2>
-     <CxPrime>0</CxPrime>
-     <Cx>0</Cx>
-     <Cy>0</Cy>
-     <focalLength>0</focalLength>
-     <hackBaseline>0</hackBaseline>
-   </plugin>
-</sensor>
-</gazebo>
+    <joint name="phantomx_camera_${suffix}" type="fixed">
+        <parent link="MP_BODY"/>
+        <child link="camera_${suffix}"/>
+        <origin xyz="${xyz}" rpy="${rpy}" />
+    </joint>
+    <link name="camera_${suffix}">
+        <inertial>
+            <origin xyz="0 0 0" rpy="0 0 0"/>
+            <mass value="0.1"/>
+            <inertia ixx="0.2" ixy="0" ixz="0" iyy="0.2" iyz="0"
+                izz="0.2"/>
+        </inertial>
+        <collision>
+            <origin xyz="0 0 0" rpy="0 0 0"/>
+            <geometry>
+                <box size="0.073000 0.276000 0.072000"/>
+            </geometry>
+        </collision>
+        <visual>
+            <origin xyz="0 0 0" rpy="0 0 0"/>
+            <geometry>
+                <!--<box size="0.073000 0.276000 0.072000"/>-->
+                <mesh filename="package://phantomx_description/meshes/kinect/meshes/kinect.dae" />
+            </geometry>
+        </visual>
+    </link>
+    <gazebo reference="camera_${suffix}">
+        <sensor name="camera_{suffix}" type="depth">
+            <update_rate>20</update_rate>
+            <camera>
+                <horizontal_fov>1.047198</horizontal_fov>
+                <image>
+                    <width>640</width>
+                    <height>480</height>
+                    <format>R8G8B8</format>
+                </image>
+                <clip>
+                    <near>0.05</near>
+                    <far>10</far>
+                </clip>
+            </camera>
+            <plugin name="camera_plugin" filename="libgazebo_ros_openni_kinect.so">
+                <baseline>0.2</baseline>
+                <alwaysOn>true</alwaysOn>
+                <updateRate>0.0</updateRate>
+                <cameraName>camera_${suffix}</cameraName>
+                <imageTopicName>/phantomx/camera_${suffix}/color/image_raw</imageTopicName>
+                <cameraInfoTopicName>/phantomx/camera_${suffix}/color/camera_info</cameraInfoTopicName>
+                <depthImageTopicName>/phantomx/camera_${suffix}/depth/image_raw</depthImageTopicName>
+                <depthImageCameraInfoTopicName>/phantomx/camera_${suffix}/depth/camera_info</depthImageCameraInfoTopicName>
+                <pointCloudTopicName>/phantomx/camera_${suffix}/depth/points</pointCloudTopicName>
+                <frameName>camera_${suffix}</frameName>
+                <pointCloudCutoff>0.1</pointCloudCutoff>
+                <pointCloudCutoffMax>2.0</pointCloudCutoffMax>
+                <distortionK1>0</distortionK1>
+                <distortionK2>0</distortionK2>
+                <distortionK3>0</distortionK3>
+                <distortionT1>0</distortionT1>
+                <distortionT2>0</distortionT2>
+                <CxPrime>0</CxPrime>
+                <Cx>0</Cx>
+                <Cy>0</Cy>
+                <focalLength>0</focalLength>
+                <hackBaseline>0</hackBaseline>
+            </plugin>
+        </sensor>
+    </gazebo>
 </xacro:macro>
     <xacro:macro name="leg_l" params="xyz rpy suffix">
@@ -381,36 +406,4 @@
     </link>
     <gazebo reference="light_link">
-        <light name='light_source_right' type='spot'>
-            <pose frame=''>0 0.03 0.03 2. 0 0</pose>
-            <id>light_source</id>
-            <attenuation>
-                <range>30</range>
-                <linear>0.005</linear>
-            </attenuation>
-            <diffuse>1 1 1 0</diffuse>
-            <specular>1 0 0 1</specular>
-            <spot>
-                <inner_angle>1</inner_angle>
-                <outer_angle>2</outer_angle>
-                <falloff>1</falloff>
-            </spot>
-            <direction>0 0 -1</direction>
-        </light>
-        <light name='light_source_left' type='spot'>
-            <pose frame=''>0  -0.03 0.03 -2. 0 0</pose>
-            <id>light_source</id>
-            <attenuation>
-                <range>30</range>
-                <linear>0.005</linear>
-            </attenuation>
-            <diffuse>1 1 1 1</diffuse>
-            <specular>1 0 0 1</specular>
-            <spot>
-                <inner_angle>1</inner_angle>
-                <outer_angle>2</outer_angle>
-                <falloff>1</falloff>
-            </spot>
-            <direction>0 0 -1</direction>
-        </light>
         <light name='light_source_front' type='spot'>
             <pose frame=''>0.1 0 0.03 0 -2. 0</pose>
@@ -431,17 +424,5 @@
         <plugin name='light_control' filename='libFlashLightPlugin.so'>
             <enable>true</enable>
-            <light>
-                <id>cylinder/light_source_right</id>
-                <duration>1</duration>
-                <interval>0</interval>
-                <color>1 1 1</color>
-            </light>
-            <light>
-                <id>cylinder/light_source_left</id>
-                <duration>1</duration>
-                <interval>0</interval>
-                <color>1 1 1</color>
-            </light>
-            <light>
+           <light>
                 <id>cylinder/light_source_front</id>
                 <duration>1</duration>
@@ -466,5 +447,5 @@
             </scan>
             <range>
-              <min>0.10</min>
+              <min>0.20</min>
               <max>15.0</max>
               <resolution>0.01</resolution>
